Commit message: Updated URDF for New Motor

File: leg_sim/urdf/one_leg_basic.urdf (robot description, URDF)
Before this commit: robot one_leg_basic, 9 links, 8 joints
Links:
- link h_motor: mass 0.511 -> 0.6; geometry collision cylinder length=0.027 radius=0.048; visual cylinder length=0.027 radius=0.048
- link l_motor: mass 0.511 -> 0.6; geometry collision cylinder length=0.027 radius=0.048; visual cylinder length=0.027 radius=0.048
- link lower_leg_link: mass 0.12 -> 0.25; geometry collision box size=0.25 0.05 0.02; visual box size=0.25 0.03 0.02
- link thigh_link: mass 0.15 -> 0.25; geometry collision box size=0.27 0.05 0.02; visual box size=0.27 0.05 0.02
Joints:
- joint body_l_motor_joint: origin xyz=0 0.011 -0.044 rpy=1.57075 0 0 -> xyz=0 0.0215 -0.058 rpy=1.57075 0 0
- joint foot_joint: origin xyz=-0.16 0 0 rpy=0 0 0 -> xyz=-0.25 0 0 rpy=0 0 0
- joint h_joint: origin xyz=0 0 -0.034 rpy=0 0 0 -> xyz=0 0 -0.0235 rpy=0 0 0
- joint l_joint: origin xyz=0 0 -0.034 rpy=0 0 0 -> xyz=0 0 -0.0235 rpy=0 0 0
- joint thigh_h_motor_joint: origin xyz=-0.16 0 0.013 rpy=0 0 0 -> xyz=-0.25 0 0 rpy=0 0 0

Commit message: Raised stand height

File: leg_sim/urdf/one_leg_basic.urdf (robot description, URDF)
Before this commit: robot one_leg_basic, 9 links, 8 joints
Links:
- link standing_link: geometry collision box size=0.65 0.05 0.05; visual box size=0.65 0.05 0.05
Joints:
- joint robot_base_joint: origin xyz=0.4 0.05 0 rpy=0 1.57075 0 -> xyz=0.6 0.05 0 rpy=0 1.57075 0

Commit message: Doubled H Joint velocity

File: leg_sim/urdf/one_leg_basic.urdf (robot description, URDF)
Before this commit: robot one_leg_basic, 9 links, 8 joints
Joints:
- joint h_joint: limit lower=0.0 upper=3.14159 effort=1000.0 velocity=0.5 -> lower=0.0 upper=3.14159 effort=1000.0 velocity=1.0
